File: AutoISP.brd (EAGLE design)
At the start: 26.6 x 15.2 mm, 7 parts

Commit message: AutoISP 1.1, fixing reversed pins
Connections:
- net N$1: now also U$1.14; no longer U$1.11
- net N$11: now also U$1.13; no longer U$1.12
- net N$12: now also U$1.12; no longer U$1.13
- net N$13: now also U$1.11; no longer U$1.14
- net N$14: now also U$1.10; no longer U$1.15
- net N$6: now also U$1.15, U$1.9; no longer U$1.10, U$1.16
- net N$7: now also U$1.16; no longer U$1.9
Routing:
- net N$7: track 57.6 -> 36.5 mm, vias 1 -> 0
- net N$6: track 34.9 -> 51.5 mm, vias 1 -> 0
- net N$1: track 50.0 -> 34.4 mm, vias 0 -> 1
- net N$12: track 12.1 -> 8.46 mm
- net N$11: track 12.7 -> 14.7 mm
- net N$5: track 20.9 -> 22.1 mm
- net N$8: track 14.2 -> 15.3 mm, vias 1 -> 0
- net N$13: track 4.36 -> 5.16 mm
Other:
- board text added: "AutoISP v1.1 µTH 2014"
- board text removed: "AutoISP v1.0 µTH 2014"

Commit message: Revise boards for better labelling and sane orientation, add AutoISP328
Parts:
- added LOGO1: OSHW-LOGOS, SparkFun-Aesthetics:OSHW-LOGO-S
- moved R1 2.84 mm to (3.81, 14.0), turned to 180 degrees
- moved BOARD 2.29 mm to (18.5, 5.71)
- moved MCU 2.29 mm to (18.5, 10.8)
- moved R2 1.80 mm to (7.37, 14.0), turned to 180 degrees
- moved LED1 1.27 mm to (12.7, 14.0)
- moved PROG 0.64 mm to (1.78, 6.99)
- moved U$1 0.64 mm to (12.7, 8.26)
Routing:
- net N$6: track 51.5 -> 30.0 mm
- net N$5: track 22.1 -> 17.3 mm, vias 1 -> 0
- net N$7: track 36.5 -> 31.8 mm
- net N$12: track 8.46 -> 12.5 mm, vias 0 -> 1
- net N$11: track 14.7 -> 10.9 mm
- net N$8: track 15.3 -> 12.4 mm, vias 0 -> 1
- net N$1: track 34.4 -> 32.5 mm, vias 1 -> 2
- net N$9: track 11.2 -> 9.39 mm
- net N$10: track 14.2 -> 12.5 mm
Other:
- board size 26.6 x 15.2 mm -> 27.9 x 16.5 mm
- board text added: "*"
- board text added: "AutoISP v1.2"
- board text added: "µTH '15 CC BY"
- board text removed: "AutoISP v1.1 µTH 2014"

Commit message: AutoISP85 1.3 (Fix flipped pin header) Add BOM
Parts:
- removed LOGO1: OSHW-LOGOS, SparkFun-Aesthetics:OSHW-LOGO-S
- added U$2: (no value), Boxtec-veclogo:ROBOXTEC-VECLOGO-NANO
- added U$3: (no value), SparkFun-Aesthetics:OSHW-LOGO-S
- R2: value (none) -> 1kΩ
- moved BOARD 0.63 mm to (18.5, 6.35)
- moved MCU 0.63 mm to (18.5, 11.4)
Routing:
- net N$9: track 9.39 -> 24.3 mm
- net N$8: track 12.4 -> 24.1 mm, vias 1 -> 0
- net N$6: track 30.0 -> 39.8 mm, vias 0 -> 1
- net N$5: track 17.3 -> 26.9 mm
- net N$7: track 31.8 -> 39.4 mm
- net N$12: track 12.5 -> 14.7 mm, vias 1 -> 0
- net N$4: track 6.34 -> 8.14 mm
- net N$1: track 32.5 -> 33.9 mm
- net N$3: track 15.4 -> 16.7 mm
- net N$14: track 7.77 -> 8.54 mm
- net N$13: track 5.02 -> 5.72 mm
- net N$11: track 10.9 -> 11.5 mm
Other:
- board text added: "µTh '15 CC BY"
- board text removed: "µTH '15 CC BY"
