File: AutoISP.sch (EAGLE design)
At the start: 7 parts

Commit message: Revise boards for better labelling and sane orientation, add AutoISP328
Parts:
- added LOGO1: OSHW-LOGOS, SparkFun-Aesthetics:OSHW-LOGOS
Changed lines of the file:
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@@
 <?xml version="1.0" encoding="utf-8"?>
 <!DOCTYPE eagle SYSTEM "eagle.dtd">
-<eagle version="7.1.0">
+<eagle version="7.2.0">
 <drawing>
 <settings>
@@
 </classes>
 <parts>
-<part name="FRAME1" library="frames" deviceset="A5L-LOC" device=""/>
 <part name="U$1" library="Microtherion" deviceset="STMAV340TTR" device=""/>
 <part name="MCU" library="SparkFun-Connectors" deviceset="AVR_SPI_PRG_6" device="PTH"/>
@@
 <part name="LED1" library="SparkFun-LED" deviceset="LED" device="1206"/>
 <part name="R2" library="SparkFun-Passives" deviceset="RESISTOR" device="0603-RES"/>
+<part name="LOGO1" library="SparkFun-Aesthetics" deviceset="OSHW-LOGO" device="S"/>
 </parts>
 <sheets>
@@
 </plain>
 <instances>
-<instance part="FRAME1" gate="G$1" x="-12.7" y="-10.16"/>
 <instance part="U$1" gate="G$1" x="78.74" y="71.12"/>
 <instance part="MCU" gate="G$1" x="134.62" y="63.5"/>
@@
 <instance part="LED1" gate="G$1" x="43.18" y="83.82"/>
 <instance part="R2" gate="G$1" x="53.34" y="88.9"/>
+<instance part="LOGO1" gate="G$1" x="142.24" y="106.68"/>
 </instances>
 <busses>

Commit message: AutoISP85 1.3 (Fix flipped pin header) Add BOM
Parts:
- removed LOGO1: OSHW-LOGOS, SparkFun-Aesthetics:OSHW-LOGOS
- R2: value (none) -> 1kΩ
Changed lines of the file:
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@@
 <part name="R1" library="SparkFun-Passives" deviceset="RESISTOR" device="0603-RES" value="10kΩ"/>
 <part name="LED1" library="SparkFun-LED" deviceset="LED" device="1206"/>
-<part name="R2" library="SparkFun-Passives" deviceset="RESISTOR" device="0603-RES"/>
-<part name="LOGO1" library="SparkFun-Aesthetics" deviceset="OSHW-LOGO" device="S"/>
+<part name="R2" library="SparkFun-Passives" deviceset="RESISTOR" device="0603-RES" value="1kΩ"/>
 </parts>
 <sheets>
@@
 <instance part="LED1" gate="G$1" x="43.18" y="83.82"/>
 <instance part="R2" gate="G$1" x="53.34" y="88.9"/>
-<instance part="LOGO1" gate="G$1" x="142.24" y="106.68"/>
 </instances>
 <busses>
