File: AutoISP328.brd (EAGLE design)
At the start: 49.5 x 17.1 mm, 6 parts, among them J1 MCU, J2 BOARD, U1 ATMEGA328P_PDIP

Commit message: AutoISP85 1.3 (Fix flipped pin header) Add BOM
Parts:
- added U$2: (no value), Boxtec-veclogo:ROBOXTEC-VECLOGO-MICRO
- U$1: device SparkFun-Aesthetics:OSHW-LOGO-S -> SparkFun-Aesthetics:OSHW-LOGO-M
- moved U$1 1.42 mm to (46.4, 2.54)
- moved J2 0.64 mm to (40.6, 6.99)
- moved J1 0.63 mm to (40.6, 12.1)
Routing:
- net N$3: track 46.8 -> 65.6 mm
- net N$5: track 24.2 -> 13.4 mm
- net N$1: track 52.8 -> 62.2 mm
- net N$6: track 22.9 -> 27.7 mm
- net N$2: track 33.4 -> 36.9 mm, vias 1 -> 0
- net N$13: track 35.7 -> 38.4 mm
- net N$10: track 42.8 -> 40.2 mm
- net N$14: track 47.0 -> 48.8 mm
- net N$4: track 14.4 -> 13.4 mm, vias 1 -> 0
- net N$8: track 23.0 -> 23.7 mm
